Commit message: 修改x2的参数

File: resources/robots/h1/h1.urdf (robot description, URDF)
Before this commit: robot h1_description, 22 links, 21 joints
Links:
- link left_ankle_link: geometry collision mesh filename=meshes/left_ankle_link.STL; visual mesh filename=meshes/left_ankle_link.STL
- link left_elbow_link: geometry collision mesh filename=meshes/left_elbow_link.STL; visual mesh filename=meshes/left_elbow_link.STL
- link left_hip_pitch_link: geometry collision mesh filename=meshes/left_hip_pitch_link.STL; visual mesh filename=meshes/left_hip_pitch_link.STL
- link left_hip_roll_link: geometry collision mesh filename=meshes/left_hip_roll_link.STL; visual mesh filename=meshes/left_hip_roll_link.STL
- link left_hip_yaw_link: geometry visual mesh filename=meshes/left_hip_yaw_link.STL
- link left_knee_link: geometry collision mesh filename=meshes/left_knee_link.STL; visual mesh filename=meshes/left_knee_link.STL
- link left_shoulder_pitch_link: geometry collision mesh filename=meshes/left_shoulder_pitch_link.STL; visual mesh filename=meshes/left_shoulder_pitch_link.STL
- link left_shoulder_roll_link: geometry collision mesh filename=meshes/left_shoulder_roll_link.STL; visual mesh filename=meshes/left_shoulder_roll_link.STL
- link left_shoulder_yaw_link: geometry collision mesh filename=meshes/left_shoulder_yaw_link.STL; visual mesh filename=meshes/left_shoulder_yaw_link.STL
- link logo_link: geometry visual mesh filename=meshes/logo_link.STL
- link pelvis: geometry collision mesh filename=meshes/pelvis.STL; visual mesh filename=meshes/pelvis.STL
- link right_ankle_link: geometry collision mesh filename=meshes/right_ankle_link.STL; visual mesh filename=meshes/right_ankle_link.STL
- link right_elbow_link: geometry collision mesh filename=meshes/right_elbow_link.STL; visual mesh filename=meshes/right_elbow_link.STL
- link right_hip_pitch_link: geometry collision mesh filename=meshes/right_hip_pitch_link.STL; visual mesh filename=meshes/right_hip_pitch_link.STL
- link right_hip_roll_link: geometry collision mesh filename=meshes/right_hip_roll_link.STL; visual mesh filename=meshes/right_hip_roll_link.STL
- link right_hip_yaw_link: geometry visual mesh filename=meshes/right_hip_yaw_link.STL
- link right_knee_link: geometry collision mesh filename=meshes/right_knee_link.STL; visual mesh filename=meshes/right_knee_link.STL
- link right_shoulder_pitch_link: geometry collision mesh filename=meshes/right_shoulder_pitch_link.STL; visual mesh filename=meshes/right_shoulder_pitch_link.STL
- link right_shoulder_roll_link: geometry collision mesh filename=meshes/right_shoulder_roll_link.STL; visual mesh filename=meshes/right_shoulder_roll_link.STL
- link right_shoulder_yaw_link: geometry collision mesh filename=meshes/right_shoulder_yaw_link.STL; visual mesh filename=meshes/right_shoulder_yaw_link.STL
- link torso_link: geometry collision mesh filename=meshes/torso_link.STL; visual mesh filename=meshes/torso_link.STL

File: resources/robots/x2/x2.urdf (robot description, URDF)
Before this commit: robot x2, 23 links, 22 joints
Joints:
- joint L_hip_roll: limit lower=-0.349 upper=0.524 effort=45 velocity=15 -> lower=-0.349 upper=0.524 effort=60 velocity=15
- joint L_hip_yaw: limit lower=-0.7854 upper=0.7854 effort=30 velocity=10 -> lower=-0.7854 upper=0.7854 effort=60 velocity=10
- joint R_hip_roll: limit lower=-0.349 upper=0.524 effort=45 velocity=15 -> lower=-0.349 upper=0.524 effort=60 velocity=15
- joint R_hip_yaw: limit lower=-0.7854 upper=0.7854 effort=30 velocity=10 -> lower=-0.7854 upper=0.7854 effort=60 velocity=10
