Commit message: 修改x2的模型

File: resources/robots/x2/x2.urdf (robot description, URDF)
Before this commit: robot x2, 23 links, 22 joints
Links:
- link L_ankle_pitch_link: geometry collision box size=0.2 0.05 0.01; collision sphere radius=0.005
- link L_elbow_pitch_link: geometry visual mesh filename=meshes/L_elbow_pitch_link.STL
- link L_shoulder_pitch_link: geometry visual mesh filename=meshes/L_shoulder_pitch_link.STL
- link L_shoulder_roll_link: geometry visual mesh filename=meshes/L_shoulder_roll_link.STL
- link L_shoulder_yaw_link: geometry visual mesh filename=meshes/L_shoulder_yaw_link.STL
- link R_ankle_pitch_link: geometry collision box size=0.2 0.05 0.01; collision sphere radius=0.005
- link R_elbow_pitch_link: geometry visual mesh filename=meshes/R_elbow_pitch_link.STL
- link R_shoulder_pitch_link: geometry visual mesh filename=meshes/R_shoulder_pitch_link.STL
- link R_shoulder_roll_link: geometry visual mesh filename=meshes/R_shoulder_roll_link.STL
- link R_shoulder_yaw_link: geometry visual mesh filename=meshes/R_shoulder_yaw_link.STL
- link head_link: geometry visual mesh filename=meshes/head_link.STL
- link logo_link: geometry visual mesh filename=meshes/logo_link.STL
- link waist_yaw_link: geometry visual mesh filename=meshes/waist_yaw_link.STL

Commit message: 删除不必要的文件

File: resources/robots/x2/x2.urdf (robot description, URDF)
Before this commit: robot x2, 23 links, 22 joints
Links:
- link L_hip_roll_link: geometry collision mesh filename=meshes/L_hip_roll_link.STL; visual mesh filename=meshes/L_hip_roll_link.STL
- link R_hip_roll_link: geometry collision mesh filename=meshes/R_hip_roll_link.STL; visual mesh filename=meshes/R_hip_roll_link.STL

Commit message: 加入tita双轮足的训练代码

File: resources/robots/x2/x2.urdf (robot description, URDF)
Before this commit: robot x2, 23 links, 22 joints
Joints:
- joint L_ankle_pitch: limit lower=-1.2217 upper=1.2217 effort=30 velocity=10 -> lower=-1.2217 upper=1.2217 effort=40 velocity=10
- joint L_hip_pitch: limit lower=-0.526 upper=2.4434 effort=60 velocity=20 -> lower=-0.526 upper=2.4434 effort=100 velocity=20
- joint L_hip_roll: limit lower=-0.349 upper=0.524 effort=60 velocity=15 -> lower=-0.349 upper=0.524 effort=100 velocity=15
- joint L_hip_yaw: limit lower=-0.7854 upper=0.7854 effort=60 velocity=10 -> lower=-0.7854 upper=0.7854 effort=100 velocity=10
- joint L_knee_pitch: limit lower=-2.3561 upper=0 effort=60 velocity=20 -> lower=-2.3561 upper=0 effort=150 velocity=20
- joint R_ankle_pitch: limit lower=-1.2217 upper=1.2217 effort=30 velocity=10 -> lower=-1.2217 upper=1.2217 effort=40 velocity=10
- joint R_hip_pitch: limit lower=-0.526 upper=2.4434 effort=60 velocity=20 -> lower=-0.526 upper=2.4434 effort=100 velocity=20
- joint R_hip_roll: limit lower=-0.349 upper=0.524 effort=60 velocity=15 -> lower=-0.349 upper=0.524 effort=100 velocity=15
- joint R_hip_yaw: limit lower=-0.7854 upper=0.7854 effort=60 velocity=10 -> lower=-0.7854 upper=0.7854 effort=100 velocity=10
- joint R_knee_pitch: limit lower=-2.3561 upper=0 effort=60 velocity=20 -> lower=-2.3561 upper=0 effort=150 velocity=20
